File: AkkordeonDiskant.kicad_sch (KiCad schematic)
At the start: 190 parts, among them J1 Conn_02x10_Odd_Even, SW101 SW_Cherry, SW102 SW_Cherry, SW103 SW_Cherry, SW104 SW_Cherry, SW105 SW_Cherry, SW106 SW_Cherry, SW107 SW_Cherry, SW108 SW_Cherry, SW109 SW_Cherry, SW110 SW_Cherry, SW111 SW_Cherry, SW112 SW_Cherry, SW113 SW_Cherry, SW114 SW_Cherry, SW115 SW_Cherry, SW116 SW_Cherry, SW117 SW_Cherry, SW118 SW_Cherry, SW201 SW_Cherry, SW202 SW_Cherry, SW203 SW_Cherry, SW204 SW_Cherry, SW205 SW_Cherry, SW206 SW_Cherry, SW207 SW_Cherry, SW208 SW_Cherry, SW209 SW_Cherry, SW210 SW_Cherry, SW211 SW_Cherry, SW212 SW_Cherry, SW213 SW_Cherry, SW214 SW_Cherry, SW215 SW_Cherry, SW216 SW_Cherry, SW217 SW_Cherry, SW218 SW_Cherry, SW219 SW_Cherry, SW301 SW_Cherry, SW302 SW_Cherry, SW303 SW_Cherry, SW304 SW_Cherry, SW305 SW_Cherry, SW306 SW_Cherry, SW307 SW_Cherry, SW308 SW_Cherry, SW309 SW_Cherry, SW310 SW_Cherry, SW311 SW_Cherry, SW312 SW_Cherry, SW313 SW_Cherry, SW314 SW_Cherry, SW315 SW_Cherry, SW316 SW_Cherry, SW317 SW_Cherry, SW318 SW_Cherry, SW401 SW_Cherry, SW402 SW_Cherry, SW403 SW_Cherry, SW404 SW_Cherry, SW405 SW_Cherry, SW406 SW_Cherry, SW407 SW_Cherry, SW408 SW_Cherry, SW409 SW_Cherry, SW410 SW_Cherry, SW411 SW_Cherry, SW412 SW_Cherry, SW413 SW_Cherry, SW414 SW_Cherry, SW415 SW_Cherry, SW416 SW_Cherry, SW417 SW_Cherry, SW418 SW_Cherry, SW419 SW_Cherry, SW501 SW_Cherry, SW502 SW_Cherry, SW503 SW_Cherry, SW504 SW_Cherry, SW505 SW_Cherry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

Commit message: Add files via upload
Connections:
- net +3V3: now also J1.4 (Pin_4)
Other:
- note added: "Diskant Knopfakkordeon Copyright 2025 Jürg Müller CH-5524 Nesselnbach"
Changed lines of the file:
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@@
   (junction (at 186.69 82.55) (diameter 0) (color 0 0 0 0)
   )
+  (junction (at 62.23 172.72) (diameter 0) (color 0 0 0 0)
+  )
   (junction (at 34.29 91.44) (diameter 0) (color 0 0 0 0)
   )
@@
     (stroke (width 0) (type default) (color 0 0 0 0))
   )
+  (wire (pts (xy 62.23 172.72) (xy 62.23 175.26))
+    (stroke (width 0) (type default) (color 0 0 0 0))
+  )
   (wire (pts (xy 303.53 82.55) (xy 303.53 96.52))
     (stroke (width 0) (type default) (color 0 0 0 0))
@@
     (stroke (width 0) (type default) (color 0 0 0 0))
   )
+  (text "Diskant Knopfakkordeon\nCopyright 2025 Jürg Müller\nCH-5524 Nesselnbach"
+    (at 104.14 57.15 0)
+    (effects (font (size 8 8)) (justify left bottom))
+  )
   (symbol (lib_id "JM_Library:SW_Cherry") (at 205.74 124.46 0) (unit 1)
